File: Battery/Battery.sch (KiCad schematic (older format))
At the start: 4 parts, among them SW1 SW_Push

Commit message: Baterijas_ MD1.1
Parts:
- added BT2: Battery, Battery_Holder:18650Battery, symbol Device:Battery
- added D2: RED, symbol Device:LED
- added R2: 470R, symbol Device:R_Small
- added SW2: SW_Push, symbol Switch:SW_Push
- BT1: footprint (none) -> Battery_Holder:SMTU2032
Connections:
- new net: BT2.2 (-), D2.1 (K)
- new net: D2.2 (A), R2.1
- new net: BT2.1 (+), SW2.1
- new net: R2.2, SW2.2
Changed lines of the file:
@@
 F 0 "BT1" H 5508 3686 50  0000 L CNN
 F 1 "3 V" H 5508 3595 50  0000 L CNN
-F 2 "" V 5390 3650 50  0001 C CNN
-F 3 "~" V 5390 3650 50  0001 C CNN
+F 2 "Battery_Holder:SMTU2032" V 5390 3650 50  0001 C CNN
+F 3 "https://eu.mouser.com/datasheet/2/346/SMTU2032-LF-6066.pdf" V 5390 3650 50  0001 C CNN
 	1    5390 3590
 	1    0    0    -1
@@
 Wire Wire Line
 	5390 3690 5390 3750
+$Comp
+L Switch:SW_Push SW2
+U 1 1 5F97355A
+P 6170 4260
+F 0 "SW2" H 6170 4545 50  0000 C CNN
+F 1 "SW_Push" H 6170 4454 50  0000 C CNN
+F 2 "" H 6170 4460 50  0001 C CNN
+F 3 "~" H 6170 4460 50  0001 C CNN
+	1    6170 4260
+	1    0    0    -1
+$EndComp
+Wire Wire Line
+	5350 4260 5970 4260
+$Comp
+L Device:R_Small R2
+U 1 1 5F973562
+P 6650 4260
+F 0 "R2" V 6454 4260 50  0000 C CNN
+F 1 "470R" V 6545 4260 50  0000 C CNN
+F 2 "" H 6650 4260 50  0001 C CNN
+F 3 "~" H 6650 4260 50  0001 C CNN
+	1    6650 4260
+	0    1    1    0
+$EndComp
+Wire Wire Line
+	6370 4260 6550 4260
+Wire Wire Line
+	6750 4260 6970 4260
+Wire Wire Line
+	6970 4260 6970 4520
+$Comp
+L Device:LED D2
+U 1 1 5F973554
+P 6970 4670
+F 0 "D2" V 7009 4552 50  0000 R CNN
+F 1 "RED" V 6918 4552 50  0000 R CNN
+F 2 "" H 6970 4670 50  0001 C CNN
+F 3 "~" H 6970 4670 50  0001 C CNN
+	1    6970 4670
+	0    -1   -1   0
+$EndComp
+$Comp
+L Device:Battery BT2
+U 1 1 5F973B4B
+P 5350 4570
+F 0 "BT2" H 5458 4616 50  0000 L CNN
+F 1 "Battery" H 5458 4525 50  0000 L CNN
+F 2 "Battery_Holder:18650Battery" V 5350 4630 50  0001 C CNN
+F 3 "~" V 5350 4630 50  0001 C CNN
+	1    5350 4570
+	1    0    0    -1
+$EndComp
+Wire Wire Line
+	5350 4370 5350 4260
+Wire Wire Line
+	5350 4770 5350 4820
+Wire Wire Line
+	5350 4820 6970 4820
 $EndSCHEMATC
