File: Single_transistor_AMP/Single_transistor_AMP.kicad_pcb (KiCad board)
At the start: 2 copper layers, 76.5 x 32.3 mm, 15 parts, among them J1 ETB06, J2 Power, Q1 2N3904, Q2 2N3904

Commit message: MD savienojumi
Parts:
- moved C5 4.00 mm to (210.6, 112.7)
- moved R4 3.20 mm to (206.9, 112.8)
- moved Re1 0.55 mm to (190.7, 110.5)
Routing:
- net +12V: track 0.00 -> 52.7 mm
- net Net-(C1-Pad2): track 0.00 -> 14.8 mm
- net Net-(C5-Pad2): track 0.00 -> 13.6 mm
- net Net-(C2-Pad1): track 0.00 -> 12.7 mm
- net Net-(C1-Pad1): track 0.00 -> 10.0 mm
- net Net-(C2-Pad2): track 0.00 -> 8.69 mm
- net Net-(C5-Pad1): track 0.00 -> 7.96 mm
- net Net-(C3-Pad1): track 0.00 -> 5.96 mm
- added copper zone on B.Cu, net GND
- added copper zone on F.Cu, net GND
Other:
- board size 76.5 x 32.3 mm -> 76.2 x 32.2 mm
Changed lines of the file:
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@@
   (general
     (thickness 1.6)
-    (drawings 9)
-    (tracks 0)
+    (drawings 12)
+    (tracks 37)
     (zones 0)
     (modules 15)
@@
   )
   (setup
-    (last_trace_width 0.25)
+    (last_trace_width 0.6)
+    (user_trace_width 0.4)
+    (user_trace_width 0.6)
     (trace_clearance 0.2)
     (zone_clearance 0.508)
@@
     (descr "Altech AK300 terminal block, pitch 5.0mm, 45 degree angled, see http://www.mouser.com/ds/2/16/PCBMETRC-24178.pdf")
     (tags "Altech AK300 terminal block pitch 5.0mm")
-    (fp_text reference J2 (at -1.92 -6.99) (layer F.SilkS)
+    (fp_text reference J2 (at 9.2 -0.55 90) (layer F.SilkS)
       (effects (font (size 1 1) (thickness 0.15)))
     )
@@
     (descr "Altech AK300 terminal block, pitch 5.0mm, 45 degree angled, see http://www.mouser.com/ds/2/16/PCBMETRC-24178.pdf")
     (tags "Altech AK300 terminal block pitch 5.0mm")
-    (fp_text reference Speaker1 (at -1.92 -6.99 90) (layer F.SilkS)
+    (fp_text reference Speaker1 (at -3.7 -2.7 180) (layer F.SilkS)
       (effects (font (size 1 1) (thickness 0.15)))
     )
@@
     (descr "Altech AK300 terminal block, pitch 5.0mm, 45 degree angled, see http://www.mouser.com/ds/2/16/PCBMETRC-24178.pdf")
     (tags "Altech AK300 terminal block pitch 5.0mm")
-    (fp_text reference J1 (at -1.92 -6.99 90) (layer F.SilkS)
+    (fp_text reference J1 (at -3.6 -0.05 180) (layer F.SilkS)
       (effects (font (size 1 1) (thickness 0.15)))
     )
@@
   )
   (module Resistor_SMD:R_0805_2012Metric (layer F.Cu)
-    (at 190.1 110.6125 90)
+    (at 190.65 110.55 90)
     (descr "Resistor SMD 0805 (2012 Metric), square (rectangular) end terminal, IPC_7351 nominal, (Body size source: https://docs.google.com/spreadsheets/d/1BsfQQcO9C6DZCsRaXUlFlo91Tg2WpOkGARC1WS5S8t0/edit?usp=sharing), generated with kicad-footprint-generator")
     (tags resistor)
     (attr smd)
-    (fp_text reference Re1 (at 0 -1.65 90) (layer F.SilkS)
+    (fp_text reference Re1 (at 2.35 0.05 180) (layer F.SilkS)
       (effects (font (size 1 1) (thickness 0.15)))
     )
@@
   )
   (module Resistor_SMD:R_0805_2012Metric (layer F.Cu)
-    (at 210.1 112.8125 90)
+    (at 206.9 112.8 90)
     (descr "Resistor SMD 0805 (2012 Metric), square (rectangular) end terminal, IPC_7351 nominal, (Body size source: https://docs.google.com/spreadsheets/d/1BsfQQcO9C6DZCsRaXUlFlo91Tg2WpOkGARC1WS5S8t0/edit?usp=sharing), generated with kicad-footprint-generator")
     (tags resistor)
@@
     (descr TO-39-3)
     (tags TO-39-3)
-    (fp_text reference Q2 (at 2.54 -5.82 90) (layer F.SilkS)
+    (fp_text reference Q2 (at 8.1 -0.3 180) (layer F.SilkS)
       (effects (font (size 1 1) (thickness 0.15)))
     )
@@
     (descr TO-39-3)
     (tags TO-39-3)
-    (fp_text reference Q1 (at 2.54 -5.82 90) (layer F.SilkS)
+    (fp_text reference Q1 (at 8.1 4.5 180) (layer F.SilkS)
       (effects (font (size 1 1) (thickness 0.15)))
     )
@@
   )
   (module Capacitor_SMD:C_0805_2012Metric (layer F.Cu)
-    (at 206.6 112.8125 90)
+    (at 210.6 112.7125 90)
     (descr "Capacitor SMD 0805 (2012 Metric), square (rectangular) end terminal, IPC_7351 nominal, (Body size source: https://docs.google.com/spreadsheets/d/1BsfQQcO9C6DZCsRaXUlFlo91Tg2WpOkGARC1WS5S8t0/edit?usp=sharing), generated with kicad-footprint-generator")
     (tags capacitor)
@@
     (tags capacitor)
     (attr smd)
-    (fp_text reference C4 (at 0 -1.65 90) (layer F.SilkS)
+    (fp_text reference C4 (at 2.2625 -0.15 180) (layer F.SilkS)
       (effects (font (size 1 1) (thickness 0.15)))
     )
@@
     (tags capacitor)
     (attr smd)
-    (fp_text reference C3 (at 0 -1.65 90) (layer F.SilkS)
+    (fp_text reference C3 (at 2.2375 -0.05 180) (layer F.SilkS)
       (effects (font (size 1 1) (thickness 0.15)))
     )
@@
     (tags "capacitor electrolytic")
     (attr smd)
-    (fp_text reference C2 (at 0 -4.35 90) (layer F.SilkS)
+    (fp_text reference C2 (at 4.15 2.1 180) (layer F.SilkS)
       (effects (font (size 1 1) (thickness 0.15)))
     )
@@
     (tags "capacitor electrolytic")
     (attr smd)
-    (fp_text reference C1 (at 0 -4.35) (layer F.SilkS)
+    (fp_text reference C1 (at 0 4.45) (layer F.SilkS)
       (effects (font (size 1 1) (thickness 0.15)))
     )
@@
     )
   )
-  (gr_line (start 222 96.35) (end 223.85 96.25) (layer Edge.Cuts) (width 0.05))
-  (gr_line (start 230.5 121) (end 230.85 103.25) (layer Edge.Cuts) (width 0.05))
+  (gr_arc (start 226.5 111.05) (end 230.5 111.05) (angle -90) (layer Edge.Cuts) (width 0.05))
+  (gr_line (start 230.5 121) (end 230.5 111.05) (layer Edge.Cuts) (width 0.05))
+  (gr_line (start 161.45 96.35) (end 179.95 96.35) (layer Edge.Cuts) (width 0.05))
+  (gr_line (start 184.1 107.05) (end 226.5 107.05) (layer Edge.Cuts) (width 0.05))
+  (gr_arc (start 184.1 106.05) (end 183.1 106.05) (angle -90) (layer Edge.Cuts) (width 0.05))
+  (gr_line (start 183.1 99.5) (end 183.1 106.05) (layer Edge.Cuts) (width 0.05))
+  (gr_arc (start 179.95 99.5) (end 183.1 99.5) (angle -90) (layer Edge.Cuts) (width 0.05))
   (gr_line (start 161.35 128.6) (end 223.5 128) (layer Edge.Cuts) (width 0.05))
-  (gr_line (start 161.45 96.35) (end 222 96.35) (layer Edge.Cuts) (width 0.05))
   (gr_line (start 154.35 121.6) (end 154.45 103.35) (layer Edge.Cuts) (width 0.05))
   (gr_arc (start 161.45 103.35) (end 161.45 96.35) (angle -90) (layer Edge.Cuts) (width 0.05))
   (gr_arc (start 161.35 121.6) (end 154.35 121.6) (angle -90) (layer Edge.Cuts) (width 0.05))
   (gr_arc (start 223.5 121) (end 223.5 128) (angle -90) (layer Edge.Cuts) (width 0.05))
-  (gr_arc (start 223.85 103.25) (end 230.85 103.25) (angle -90) (layer Edge.Cuts) (width 0.05))
+  (segment (start 179.6 117.25) (end 181.45 115.4) (width 0.6) (layer F.Cu) (net 1))
+  (segment (start 178.2 117.25) (end 179.6 117.25) (width 0.6) (layer F.Cu) (net 1))
+  (segment (start 179.7 117.25) (end 181.45 119) (width 0.6) (layer F.Cu) (net 1))
+  (segment (start 178.2 117.25) (end 179.7 117.25) (width 0.6) (layer F.Cu) (net 1))
+  (segment (start 183.06 117.39) (end 181.45 119) (width 0.6) (layer F.Cu) (net 1))
+  (segment (start 187.61 117.39) (end 183.06 117.39) (width 0.6) (layer F.Cu) (net 1))
+  (segment (start 163.15 117.25) (end 162.75 116.85) (width 0.6) (layer F.Cu) (net 2))
+  (segment (start 172.6 117.25) (end 163.15 117.25) (width 0.6) (layer F.Cu) (net 2))
+  (segment (start 203.82 116.85) (end 206.56 119.59) (width 0.6) (layer F.Cu) (net 3))
+  (segment (start 199 116.85) (end 203.82 116.85) (width 0.6) (layer F.Cu) (net 3))
+  (segment (start 191.1 122.45) (end 190.15 123.4) (width 0.6) (layer F.Cu) (net 4))
+  (segment (start 199 122.45) (end 191.1 122.45) (width 0.6) (layer F.Cu) (net 4))
+  (segment (start 190.15 119.93) (end 190.15 123.4) (width 0.6) (layer F.Cu) (net 4))
+  (segment (start 190.65 114.35) (end 190.15 114.85) (width 0.6) (layer F.Cu) (net 6))
+  (segment (start 190.65 111.4875) (end 190.65 114.35) (width 0.6) (layer F.Cu) (net 6))
+  (segment (start 190.7375 111.575) (end 190.65 111.4875) (width 0.6) (layer F.Cu) (net 6))
+  (segment (start 193 111.575) (end 190.7375 111.575) (width 0.6) (layer F.Cu) (net 6))
+  (segment (start 177.1 109.175) (end 181.45 113.525) (width 0.6) (layer F.Cu) (net 7))
+  (segment (start 177.1 105.95) (end 177.1 109.175) (width 0.6) (layer F.Cu) (net 7))
+  (segment (start 183.475 111.5) (end 181.45 113.525) (width 0.6) (layer F.Cu) (net 7))
+  (segment (start 188 111.5) (end 183.475 111.5) (width 0.6) (layer F.Cu) (net 7))
+  (segment (start 188 115.15) (end 189.025 116.175) (width 0.6) (layer F.Cu) (net 7))
+  (segment (start 188 111.5) (end 188 115.15) (width 0.6) (layer F.Cu) (net 7))
+  (segment (start 189.025 116.175) (end 189.15 116.3) (width 0.25) (layer F.Cu) (net 7))
+  (segment (start 189.15 118.35) (end 187.95 119.55) (width 0.6) (layer F.Cu) (net 7))
+  (segment (start 189.15 116.3) (end 189.15 118.35) (width 0.6) (layer F.Cu) (net 7))
+  (segment (start 187.95 123.075) (end 190.15 125.275) (width 0.6) (layer F.Cu) (net 7))
+  (segment (start 187.95 119.55) (end 187.95 123.075) (width 0.6) (layer F.Cu) (net 7))
+  (segment (start 205.955 125.275) (end 209.1 122.13) (width 0.6) (layer F.Cu) (net 7))
+  (segment (start 190.15 125.275) (end 205.955 125.275) (width 0.6) (layer F.Cu) (net 7))
+  (segment (start 221.1 115.51) (end 221.1 117.1) (width 0.6) (layer F.Cu) (net 8))
+  (segment (start 217.365 111.775) (end 221.1 115.51) (width 0.6) (layer F.Cu) (net 8))
+  (segment (start 210.6 111.775) (end 217.365 111.775) (width 0.6) (layer F.Cu) (net 8))
+  (segment (start 206.9 114.85) (end 209.1 117.05) (width 0.6) (layer F.Cu) (net 9))
+  (segment (start 206.9 113.7375) (end 206.9 114.85) (width 0.6) (layer F.Cu) (net 9))
+  (segment (start 206.9875 113.65) (end 206.9 113.7375) (width 0.6) (layer F.Cu) (net 9))
+  (segment (start 210.6 113.65) (end 206.9875 113.65) (width 0.6) (layer F.Cu) (net 9))
+  (zone (net 5) (net_name GND) (layer B.Cu) (hatch edge 0.508)
+    (connect_pads (clearance 0.508))
+    (min_thickness 0.254)
+    (fill (arc_segments 32) (thermal_gap 0.508) (thermal_bridge_width 0.508))
+    (polygon
+      (pts
+        (xy 156 125.65) (xy 156 99) (xy 182.8 98.95) (xy 182.8 107.65) (xy 228 107.65)
+        (xy 228 125.95) (xy 156 125.95)
+      )
+    )
+  )
+  (zone (net 5) (net_name GND) (layer F.Cu) (hatch edge 0.508)
+    (connect_pads (clearance 0.508))
+    (min_thickness 0.254)
+    (fill (arc_segments 32) (thermal_gap 0.508) (thermal_bridge_width 0.508))
+    (polygon
+      (pts
+        (xy 156 125.95) (xy 156 99) (xy 182.8 98.95) (xy 182.8 107.65) (xy 227.95 107.65)
+        (xy 228 107.65) (xy 228 125.95)
+      )
+    )
+  )
 )
