File: Single_transistor_AMP/Single_transistor_AMP.sch (KiCad schematic (older format))
At the start: 14 parts, among them J1 ETB06, Q1 2N3904, Q2 2N3904

Commit message: Pedejais MD
Parts:
- J1: footprint TerminalBlock:TerminalBlock_bornier-2_P3.5mm -> TerminalBlock:TerminalBlock_Altech_AK300-2_P5.00mm
- Speaker1: renamed from Speaker; footprint TerminalBlock:TerminalBlock_bornier-2_P3.5mm -> TerminalBlock:TerminalBlock_Altech_AK300-2_P5.00mm
- renumbered Re to Re1
Changed lines of the file:
@@
 $EndComp
 $Comp
-L Device:R_Small Re
+L Device:R_Small Re1
 U 1 1 5F872D97
 P 2775 3340
-F 0 "Re" H 2834 3431 50  0000 L CNN
+F 0 "Re1" H 2834 3431 50  0000 L CNN
 F 1 "470" H 2834 3340 50  0000 L CNN
 F 2 "Resistor_SMD:R_0805_2012Metric" H 2775 3340 50  0001 C CNN
@@
 $EndComp
 $Comp
-L power:+12V #PWR?
+L power:+12V #PWR0101
 U 1 1 5F87C097
 P 2470 2375
-F 0 "#PWR?" H 2470 2225 50  0001 C CNN
+F 0 "#PWR0101" H 2470 2225 50  0001 C CNN
 F 1 "+12V" H 2485 2548 50  0000 C CNN
 F 2 "Connector_Pin:Pin_D1.0mm_L10.0mm" H 2470 2375 50  0001 C CNN
@@
 $EndComp
 $Comp
-L power:GND #PWR?
+L power:GND #PWR0102
 U 1 1 5F87CC2B
 P 2120 3605
-F 0 "#PWR?" H 2120 3355 50  0001 C CNN
+F 0 "#PWR0102" H 2120 3355 50  0001 C CNN
 F 1 "GND" H 2125 3432 50  0000 C CNN
 F 2 "" H 2120 3605 50  0001 C CNN
@@
 $EndComp
 $Comp
-L power:GND #PWR?
+L power:GND #PWR0103
 U 1 1 5F87E8D8
 P 2775 3570
-F 0 "#PWR?" H 2775 3320 50  0001 C CNN
+F 0 "#PWR0103" H 2775 3320 50  0001 C CNN
 F 1 "GND" H 2780 3397 50  0000 C CNN
 F 2 "" H 2775 3570 50  0001 C CNN
@@
 F 0 "J1" H 948 3100 50  0000 C CNN
 F 1 "ETB06" H 948 2741 50  0001 C CNN
-F 2 "TerminalBlock:TerminalBlock_bornier-2_P3.5mm" H 1030 2975 50  0001 C CNN
+F 2 "TerminalBlock:TerminalBlock_Altech_AK300-2_P5.00mm" H 1030 2975 50  0001 C CNN
 F 3 "https://www.us-electronics.com/files/TerminalBlocks.pdf" H 1030 2975 50  0001 C CNN
 	1    1030 2975
@@
 	1230 2975 1535 2975
 $Comp
-L power:GND #PWR?
+L power:GND #PWR0104
 U 1 1 5F887ED9
 P 1230 3210
-F 0 "#PWR?" H 1230 2960 50  0001 C CNN
+F 0 "#PWR0104" H 1230 2960 50  0001 C CNN
 F 1 "GND" H 1235 3037 50  0000 C CNN
 F 2 "" H 1230 3210 50  0001 C CNN
@@
 	4105 2380 4105 2375
 $Comp
-L power:GND #PWR?
+L power:GND #PWR0105
 U 1 1 5F89682F
 P 4705 2750
-F 0 "#PWR?" H 4705 2500 50  0001 C CNN
+F 0 "#PWR0105" H 4705 2500 50  0001 C CNN
 F 1 "GND" H 4710 2577 50  0000 C CNN
 F 2 "" H 4705 2750 50  0001 C CNN
@@
 	4105 3270 4105 2945
 $Comp
-L power:GND #PWR?
+L power:GND #PWR0106
 U 1 1 5F899C24
 P 4105 3785
-F 0 "#PWR?" H 4105 3535 50  0001 C CNN
+F 0 "#PWR0106" H 4105 3535 50  0001 C CNN
 F 1 "GND" H 4110 3612 50  0000 C CNN
 F 2 "" H 4105 3785 50  0001 C CNN
@@
 	2775 3195 2775 3175
 $Comp
-L power:GND #PWR?
+L power:GND #PWR0107
 U 1 1 5F86C8E9
 P 3150 3635
-F 0 "#PWR?" H 3150 3385 50  0001 C CNN
+F 0 "#PWR0107" H 3150 3385 50  0001 C CNN
 F 1 "GND" H 3155 3462 50  0000 C CNN
 F 2 "" H 3150 3635 50  0001 C CNN
@@
 	3150 3635 3150 3550
 $Comp
-L Device:Speaker Speaker
+L Device:Speaker Speaker1
 U 1 1 5F86E00F
 P 4995 3570
-F 0 "Speaker" H 5165 3566 50  0000 L CNN
+F 0 "Speaker1" H 5165 3566 50  0000 L CNN
 F 1 "8 ohm " H 5165 3475 50  0000 L CNN
-F 2 "TerminalBlock:TerminalBlock_bornier-2_P3.5mm" H 4995 3370 50  0001 C CNN
+F 2 "TerminalBlock:TerminalBlock_Altech_AK300-2_P5.00mm" H 4995 3370 50  0001 C CNN
 F 3 "http://www.farnell.com/datasheets/1936659.pdf?_ga=2.155260091.1437130079.1602656322-238660856.1582371978" H 4985 3520 50  0001 C CNN
 	1    4995 3570

Commit message: MD savienojumi
Parts:
- added J2: Power, TerminalBlock:TerminalBlock_Altech_AK300-2_P5.00mm, symbol Connector:Screw_Terminal_01x02
- R1: footprint http://www.farnell.com/datasheets/2710384.pdf?_ga=2.48968486.1437130079.1602656322-238660856.1582371978 -> Resistor_SMD:R_0805_2012Metric
Connections:
- net +12V: now also J2.1 (Pin_1)
- net GND: now also J2.2 (Pin_2)
Changed lines of the file:
@@
 F 0 "R1" H 2179 2796 50  0000 L CNN
 F 1 "1K1" H 2179 2705 50  0000 L CNN
-F 2 "http://www.farnell.com/datasheets/2710384.pdf?_ga=2.48968486.1437130079.1602656322-238660856.1582371978" H 2120 2705 50  0001 C CNN
+F 2 "Resistor_SMD:R_0805_2012Metric" H 2120 2705 50  0001 C CNN
 F 3 "~" H 2120 2705 50  0001 C CNN
 F 4 "100 mW" V 2050 2550 50  0000 L CNN "Max Power"
@@
 Wire Wire Line
 	4795 3670 4795 3710
+$Comp
+L Connector:Screw_Terminal_01x02 J2
+U 1 1 5FB45609
+P 3870 4595
+F 0 "J2" H 3788 4720 50  0000 C CNN
+F 1 "Power" H 3788 4361 50  0001 C CNN
+F 2 "TerminalBlock:TerminalBlock_Altech_AK300-2_P5.00mm" H 3870 4595 50  0001 C CNN
+F 3 "https://www.us-electronics.com/files/TerminalBlocks.pdf" H 3870 4595 50  0001 C CNN
+	1    3870 4595
+	1    0    0    1
+$EndComp
+$Comp
+L power:GND #PWR0108
+U 1 1 5FB45610
+P 3670 4360
+F 0 "#PWR0108" H 3670 4110 50  0001 C CNN
+F 1 "GND" H 3675 4187 50  0000 C CNN
+F 2 "" H 3670 4360 50  0001 C CNN
+F 3 "" H 3670 4360 50  0001 C CNN
+	1    3670 4360
+	-1   0    0    1
+$EndComp
+Wire Wire Line
+	3670 4360 3670 4495
+$Comp
+L power:+12V #PWR0109
+U 1 1 5FB469A1
+P 3640 4645
+F 0 "#PWR0109" H 3640 4495 50  0001 C CNN
+F 1 "+12V" H 3655 4818 50  0000 C CNN
+F 2 "Connector_Pin:Pin_D1.0mm_L10.0mm" H 3640 4645 50  0001 C CNN
+F 3 "" H 3640 4645 50  0001 C CNN
+	1    3640 4645
+	-1   0    0    1
+$EndComp
+Wire Wire Line
+	3640 4645 3640 4595
+Wire Wire Line
+	3640 4595 3670 4595
 $EndSCHEMATC
