File: TDA7491/TDA7491 OP AMP/TDA7491 OP AMP.kicad_pcb (KiCad board)
At the start: 2 copper layers, 99 x 93 mm, 67 parts, among them IC2 3V3, J1 Signal, J2 L-output, J3 R-output, J4 Power 12V, Q1 npn, Q2 npn, U1 TDA7491, U2 DFplayermini, U3 Bluetooth, U4 5V_stabilizators

Commit message: Add files via upload
Routing:
- net Audio_input-: track 67.0 -> 77.4 mm
- net Net-(R1-Pad1): track 15.9 -> 17.5 mm
- net B.T.Rx: track 57.9 -> 57.1 mm
